File: meteo_station/meteo_station.kicad_sch (KiCad schematic)
At the start: 9 parts, among them SW1 SW_SPDT, U1 TP4056, U2 ESP32-WROOM, U3 DS18B20, U4 BH1750, U5 BME280

Commit message: Fixes
Parts:
- added R1, R2: 4.7K, symbol Device:R
- renumbered R1 to R3
Connections:
- net 3V3: now also R1.1, R2.1
- net SCL: now also R1.2
- net SDA: now also R2.2
Other:
- note added: "OPTIONAL I2C PULL UP"
Changed lines of the file:
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@@
   (no_connect (at 99.06 60.96))
   (no_connect (at 116.84 73.66))
+  (polyline (pts (xy 26.67 97.79) (xy 26.67 120.65))
+    (stroke (width 0) (type default) (color 0 0 0 0))
+  )
   (wire (pts (xy 146.05 71.12) (xy 146.05 78.74))
     (stroke (width 0) (type default) (color 0 0 0 0))
@@
     (stroke (width 0) (type default) (color 0 0 0 0))
   )
+  (polyline (pts (xy 26.67 97.79) (xy 73.66 97.79))
+    (stroke (width 0) (type default) (color 0 0 0 0))
+  )
+  (wire (pts (xy 38.1 114.3) (xy 45.72 114.3))
+    (stroke (width 0) (type default) (color 0 0 0 0))
+  )
   (wire (pts (xy 154.94 48.26) (xy 156.21 48.26))
     (stroke (width 0) (type default) (color 0 0 0 0))
@@
     (stroke (width 0) (type default) (color 0 0 0 0))
   )
+  (wire (pts (xy 38.1 104.14) (xy 45.72 104.14))
+    (stroke (width 0) (type default) (color 0 0 0 0))
+  )
   (wire (pts (xy 87.63 44.45) (xy 87.63 90.17))
     (stroke (width 0) (type default) (color 0 0 0 0))
@@
     (stroke (width 0) (type default) (color 0 0 0 0))
   )
+  (wire (pts (xy 53.34 104.14) (xy 62.23 104.14))
+    (stroke (width 0) (type default) (color 0 0 0 0))
+  )
   (wire (pts (xy 137.16 52.07) (xy 137.16 53.34))
     (stroke (width 0) (type default) (color 0 0 0 0))
@@
     (stroke (width 0) (type default) (color 0 0 0 0))
   )
+  (polyline (pts (xy 26.67 120.65) (xy 73.66 120.65))
+    (stroke (width 0) (type default) (color 0 0 0 0))
+  )
   (wire (pts (xy 69.85 57.15) (xy 73.66 57.15))
     (stroke (width 0) (type default) (color 0 0 0 0))
@@
     (stroke (width 0) (type default) (color 0 0 0 0))
   )
+  (polyline (pts (xy 73.66 120.65) (xy 73.66 97.79))
+    (stroke (width 0) (type default) (color 0 0 0 0))
+  )
   (wire (pts (xy 116.84 83.82) (xy 116.84 90.17))
     (stroke (width 0) (type default) (color 0 0 0 0))
@@
     (stroke (width 0) (type default) (color 0 0 0 0))
   )
+  (wire (pts (xy 53.34 114.3) (xy 62.23 114.3))
+    (stroke (width 0) (type default) (color 0 0 0 0))
+  )
   (wire (pts (xy 154.94 49.53) (xy 154.94 48.26))
     (stroke (width 0) (type default) (color 0 0 0 0))
@@
   (wire (pts (xy 66.04 58.42) (xy 66.04 46.99))
     (stroke (width 0) (type default) (color 0 0 0 0))
+  )
+  (text "OPTIONAL I2C PULL UP" (at 26.67 96.52 0)
+    (effects (font (size 1.27 1.27)) (justify left bottom))
+  )
+  (global_label "SCL" (shape input) (at 38.1 104.14 180) (fields_autoplaced)
+    (effects (font (size 1.27 1.27)) (justify right))
+    (property "Intersheet References" "${INTERSHEET_REFS}" (id 0) (at 32.1793 104.2194 0)
+      (effects (font (size 1.27 1.27)) (justify right) hide)
+    )
+  )
+  (global_label "3V3" (shape input) (at 62.23 114.3 0) (fields_autoplaced)
+    (effects (font (size 1.27 1.27)) (justify left))
+    (property "Intersheet References" "${INTERSHEET_REFS}" (id 0) (at 68.1507 114.2206 0)
+      (effects (font (size 1.27 1.27)) (justify left) hide)
+    )
+  )
+  (global_label "SDA" (shape input) (at 38.1 114.3 180) (fields_autoplaced)
+    (effects (font (size 1.27 1.27)) (justify right))
+    (property "Intersheet References" "${INTERSHEET_REFS}" (id 0) (at 32.1188 114.3794 0)
+      (effects (font (size 1.27 1.27)) (justify right) hide)
+    )
   )
   (global_label "3V3" (shape input) (at 148.59 95.25 180) (fields_autoplaced)
@@
     )
   )
+  (global_label "3V3" (shape input) (at 62.23 104.14 0) (fields_autoplaced)
+    (effects (font (size 1.27 1.27)) (justify left))
+    (property "Intersheet References" "${INTERSHEET_REFS}" (id 0) (at 68.1507 104.0606 0)
+      (effects (font (size 1.27 1.27)) (justify left) hide)
+    )
+  )
   (global_label "SCL" (shape input) (at 151.13 29.21 180) (fields_autoplaced)
     (effects (font (size 1.27 1.27)) (justify right))
@@
     )
     (pin "1")
+  )
+  (symbol (lib_id "Device:R") (at 49.53 114.3 270) (unit 1)
+    (in_bom yes) (on_board yes)
+    (property "Reference" "R2" (id 0) (at 49.53 111.76 90))
+    (property "Value" "4.7K" (id 1) (at 49.53 116.84 90))
+    (property "Footprint" "" (id 2) (at 49.53 112.522 90)
+      (effects (font (size 1.27 1.27)) hide)
+    )
+    (property "Datasheet" "~" (id 3) (at 49.53 114.3 0)
+      (effects (font (size 1.27 1.27)) hide)
+    )
+    (pin "1")
+    (pin "2")
   )
   (symbol (lib_id "power:GND") (at 137.16 27.94 0) (unit 1)
@@
     (pin "1")
   )
+  (symbol (lib_id "Device:R") (at 49.53 104.14 270) (unit 1)
+    (in_bom yes) (on_board yes)
+    (property "Reference" "R1" (id 0) (at 49.53 101.6 90))
+    (property "Value" "4.7K" (id 1) (at 49.53 106.68 90))
+    (property "Footprint" "" (id 2) (at 49.53 102.362 90)
+      (effects (font (size 1.27 1.27)) hide)
+    )
+    (property "Datasheet" "~" (id 3) (at 49.53 104.14 0)
+      (effects (font (size 1.27 1.27)) hide)
+    )
+    (pin "1")
+    (pin "2")
+  )
   (symbol (lib_id "meteo_station_symbols:DS18B20") (at 161.29 71.12 0) (mirror y) (unit 1)
     (in_bom yes) (on_board yes) (fields_autoplaced)
@@
   (symbol (lib_id "Device:R") (at 151.13 86.36 180) (unit 1)
     (in_bom yes) (on_board yes)
-    (property "Reference" "R1" (id 0) (at 154.94 87.63 0))
+    (property "Reference" "R3" (id 0) (at 154.94 87.63 0))
     (property "Value" "4.7K" (id 1) (at 154.94 85.09 0))
     (property "Footprint" "" (id 2) (at 152.908 86.36 90)
@@
       (reference "BT1") (unit 1) (value "Battery") (footprint "")
     )
+    (path "/ca4ca9b5-a17a-4638-a4ca-7ab1ae3d54a1"
+      (reference "R1") (unit 1) (value "4.7K") (footprint "")
+    )
+    (path "/23797d9f-2c0e-4299-b2b5-bbbc7f9fdf31"
+      (reference "R2") (unit 1) (value "4.7K") (footprint "")
+    )
     (path "/e6ee56a2-86c1-42e9-9f14-cd735802777f"
-      (reference "R1") (unit 1) (value "4.7K") (footprint "")
+      (reference "R3") (unit 1) (value "4.7K") (footprint "")
     )
     (path "/e3bc8b35-8aa9-44ed-b10b-bbd343541f80"

Commit message: First random assignment
Parts:
- BT1: footprint (none) -> Battery:BatteryHolder_MPD_BH-18650-PC2
- R1: footprint (none) -> Resistor_SMD:R_0603_1608Metric
- R2, R3: footprint (none) -> Resistor_SMD:R_0603_1608Metric_Pad0.98x0.95mm_HandSolder
- SC1: footprint (none) -> Connector_PinHeader_2.54mm:PinHeader_1x02_P2.54mm_Vertical
- SW1: footprint (none) -> Button_Switch_THT:SW_Slide_1P2T_CK_OS102011MS2Q
- U1, U2, U4, U5: footprint (none) -> meteo_station_footprints:BME280
Changed lines of the file:
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@@
     (property "Reference" "U1" (id 0) (at 52.07 52.07 0))
     (property "Value" "TP4056" (id 1) (at 52.07 54.61 0))
-    (property "Footprint" "" (id 2) (at 52.07 62.23 0)
+    (property "Footprint" "meteo_station_footprints:BME280" (id 2) (at 52.07 62.23 0)
       (effects (font (size 1.27 1.27)) hide)
     )
@@
     (property "Reference" "R2" (id 0) (at 49.53 111.76 90))
     (property "Value" "4.7K" (id 1) (at 49.53 116.84 90))
-    (property "Footprint" "" (id 2) (at 49.53 112.522 90)
+    (property "Footprint" "Resistor_SMD:R_0603_1608Metric_Pad0.98x0.95mm_HandSolder" (id 2) (at 49.53 112.522 90)
       (effects (font (size 1.27 1.27)) hide)
     )
@@
     (property "Reference" "U2" (id 0) (at 107.95 41.91 0))
     (property "Value" "ESP32-WROOM" (id 1) (at 107.95 44.45 0))
-    (property "Footprint" "" (id 2) (at 106.68 53.34 0)
+    (property "Footprint" "meteo_station_footprints:BME280" (id 2) (at 106.68 53.34 0)
       (effects (font (size 1.27 1.27)) hide)
     )
@@
     (property "Reference" "SW1" (id 0) (at 74.93 39.37 0))
     (property "Value" "SW_SPDT" (id 1) (at 74.93 41.91 0))
-    (property "Footprint" "" (id 2) (at 74.93 46.99 0)
+    (property "Footprint" "Button_Switch_THT:SW_Slide_1P2T_CK_OS102011MS2Q" (id 2) (at 74.93 46.99 0)
       (effects (font (size 1.27 1.27)) hide)
     )
@@
       (effects (font (size 1.27 1.27)) (justify left))
     )
-    (property "Footprint" "" (id 2) (at 73.66 60.706 90)
+    (property "Footprint" "Battery:BatteryHolder_MPD_BH-18650-PC2" (id 2) (at 73.66 60.706 90)
       (effects (font (size 1.27 1.27)) hide)
     )
@@
     (property "Reference" "R1" (id 0) (at 49.53 101.6 90))
     (property "Value" "4.7K" (id 1) (at 49.53 106.68 90))
-    (property "Footprint" "" (id 2) (at 49.53 102.362 90)
+    (property "Footprint" "Resistor_SMD:R_0603_1608Metric" (id 2) (at 49.53 102.362 90)
       (effects (font (size 1.27 1.27)) hide)
     )
@@
       (effects (font (size 1.27 1.27)) (justify left))
     )
-    (property "Footprint" "" (id 2) (at 30.48 61.976 90)
+    (property "Footprint" "Connector_PinHeader_2.54mm:PinHeader_1x02_P2.54mm_Vertical" (id 2) (at 30.48 61.976 90)
       (effects (font (size 1.27 1.27)) hide)
     )
@@
       (effects (font (size 1.27 1.27)) (justify right))
     )
-    (property "Footprint" "" (id 2) (at 163.83 19.05 0)
+    (property "Footprint" "meteo_station_footprints:BME280" (id 2) (at 163.83 19.05 0)
       (effects (font (size 1.27 1.27)) hide)
     )
@@
     (property "Reference" "R3" (id 0) (at 154.94 87.63 0))
     (property "Value" "4.7K" (id 1) (at 154.94 85.09 0))
-    (property "Footprint" "" (id 2) (at 152.908 86.36 90)
+    (property "Footprint" "Resistor_SMD:R_0603_1608Metric_Pad0.98x0.95mm_HandSolder" (id 2) (at 152.908 86.36 90)
       (effects (font (size 1.27 1.27)) hide)
     )
@@
       (effects (font (size 1.27 1.27)) (justify left))
     )
-    (property "Footprint" "" (id 2) (at 162.56 43.18 0)
+    (property "Footprint" "meteo_station_footprints:BME280" (id 2) (at 162.56 43.18 0)
       (effects (font (size 1.27 1.27)) hide)
     )
@@
     )
     (path "/a7c72c64-c327-4ae9-9904-b1572c7f32f2"
-      (reference "BT1") (unit 1) (value "Battery") (footprint "")
+      (reference "BT1") (unit 1) (value "Battery") (footprint "Battery:BatteryHolder_MPD_BH-18650-PC2")
     )
     (path "/ca4ca9b5-a17a-4638-a4ca-7ab1ae3d54a1"
-      (reference "R1") (unit 1) (value "4.7K") (footprint "")
+      (reference "R1") (unit 1) (value "4.7K") (footprint "Resistor_SMD:R_0603_1608Metric")
     )
     (path "/23797d9f-2c0e-4299-b2b5-bbbc7f9fdf31"
-      (reference "R2") (unit 1) (value "4.7K") (footprint "")
+      (reference "R2") (unit 1) (value "4.7K") (footprint "Resistor_SMD:R_0603_1608Metric_Pad0.98x0.95mm_HandSolder")
     )
     (path "/e6ee56a2-86c1-42e9-9f14-cd735802777f"
-      (reference "R3") (unit 1) (value "4.7K") (footprint "")
+      (reference "R3") (unit 1) (value "4.7K") (footprint "Resistor_SMD:R_0603_1608Metric_Pad0.98x0.95mm_HandSolder")
     )
     (path "/e3bc8b35-8aa9-44ed-b10b-bbd343541f80"
-      (reference "SC1") (unit 1) (value "Solar_Cell") (footprint "")
+      (reference "SC1") (unit 1) (value "Solar_Cell") (footprint "Connector_PinHeader_2.54mm:PinHeader_1x02_P2.54mm_Vertical")
     )
     (path "/a30bd64c-5664-40ec-b5dc-e115cbdaa123"
-      (reference "SW1") (unit 1) (value "SW_SPDT") (footprint "")
+      (reference "SW1") (unit 1) (value "SW_SPDT") (footprint "Button_Switch_THT:SW_Slide_1P2T_CK_OS102011MS2Q")
     )
     (path "/1916a1e3-b413-4657-ae92-e4caf1d88b76"
-      (reference "U1") (unit 1) (value "TP4056") (footprint "")
+      (reference "U1") (unit 1) (value "TP4056") (footprint "meteo_station_footprints:BME280")
     )
     (path "/93a49863-00ee-408b-9e67-37bd2abd68da"
-      (reference "U2") (unit 1) (value "ESP32-WROOM") (footprint "")
+      (reference "U2") (unit 1) (value "ESP32-WROOM") (footprint "meteo_station_footprints:BME280")
     )
     (path "/dfceaf99-0117-4f2d-8240-339c614bf0fc"
@@
     )
     (path "/ed6dd4e3-cfe6-415c-94e1-38553a3a4527"
-      (reference "U4") (unit 1) (value "BH1750") (footprint "")
+      (reference "U4") (unit 1) (value "BH1750") (footprint "meteo_station_footprints:BME280")
     )
     (path "/e68039ac-75c7-42b9-b4c3-f36337a478dc"
-      (reference "U5") (unit 1) (value "BME280") (footprint "")
-    )
-  )
+      (reference "U5") (unit 1) (value "BME280") (footprint "meteo_station_footprints:BME280")
+    )
+  )

Commit message: First draft of PCB
Parts:
- U2: footprint meteo_station_footprints:BME280 -> meteo_station_footprints:ESP32-WROOM
- U4: footprint meteo_station_footprints:BME280 -> meteo_station_footprints:BH1750
Changed lines of the file:
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@@
     (property "Reference" "U2" (id 0) (at 107.95 41.91 0))
     (property "Value" "ESP32-WROOM" (id 1) (at 107.95 44.45 0))
-    (property "Footprint" "meteo_station_footprints:BME280" (id 2) (at 106.68 53.34 0)
+    (property "Footprint" "meteo_station_footprints:ESP32-WROOM" (id 2) (at 106.68 53.34 0)
       (effects (font (size 1.27 1.27)) hide)
     )
@@
       (effects (font (size 1.27 1.27)) (justify left))
     )
-    (property "Footprint" "meteo_station_footprints:BME280" (id 2) (at 162.56 43.18 0)
+    (property "Footprint" "meteo_station_footprints:BH1750" (id 2) (at 162.56 43.18 0)
       (effects (font (size 1.27 1.27)) hide)
     )
@@
     )
     (path "/93a49863-00ee-408b-9e67-37bd2abd68da"
-      (reference "U2") (unit 1) (value "ESP32-WROOM") (footprint "meteo_station_footprints:BME280")
+      (reference "U2") (unit 1) (value "ESP32-WROOM") (footprint "meteo_station_footprints:ESP32-WROOM")
     )
     (path "/dfceaf99-0117-4f2d-8240-339c614bf0fc"
@@
     )
     (path "/ed6dd4e3-cfe6-415c-94e1-38553a3a4527"
-      (reference "U4") (unit 1) (value "BH1750") (footprint "meteo_station_footprints:BME280")
+      (reference "U4") (unit 1) (value "BH1750") (footprint "meteo_station_footprints:BH1750")
     )
     (path "/e68039ac-75c7-42b9-b4c3-f36337a478dc"

Commit message: Add some footprints
Parts:
- R2, R3: footprint Resistor_SMD:R_0603_1608Metric_Pad0.98x0.95mm_HandSolder -> Resistor_SMD:R_0603_1608Metric
- SC1: footprint Connector_PinHeader_2.54mm:PinHeader_1x02_P2.54mm_Vertical -> meteo_station_footprints:SolarPanel
- SW1: footprint Button_Switch_THT:SW_Slide_1P2T_CK_OS102011MS2Q -> meteo_station_footprints:MTS102
- U1: footprint meteo_station_footprints:BME280 -> meteo_station_footprints:TP4056
Changed lines of the file:
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@@
     (property "Reference" "U1" (id 0) (at 52.07 52.07 0))
     (property "Value" "TP4056" (id 1) (at 52.07 54.61 0))
-    (property "Footprint" "meteo_station_footprints:BME280" (id 2) (at 52.07 62.23 0)
+    (property "Footprint" "meteo_station_footprints:TP4056" (id 2) (at 52.07 62.23 0)
       (effects (font (size 1.27 1.27)) hide)
     )
@@
     (property "Reference" "R2" (id 0) (at 49.53 111.76 90))
     (property "Value" "4.7K" (id 1) (at 49.53 116.84 90))
-    (property "Footprint" "Resistor_SMD:R_0603_1608Metric_Pad0.98x0.95mm_HandSolder" (id 2) (at 49.53 112.522 90)
+    (property "Footprint" "Resistor_SMD:R_0603_1608Metric" (id 2) (at 49.53 112.522 90)
       (effects (font (size 1.27 1.27)) hide)
     )
@@
     (property "Reference" "SW1" (id 0) (at 74.93 39.37 0))
     (property "Value" "SW_SPDT" (id 1) (at 74.93 41.91 0))
-    (property "Footprint" "Button_Switch_THT:SW_Slide_1P2T_CK_OS102011MS2Q" (id 2) (at 74.93 46.99 0)
+    (property "Footprint" "meteo_station_footprints:MTS102" (id 2) (at 74.93 46.99 0)
       (effects (font (size 1.27 1.27)) hide)
     )
@@
       (effects (font (size 1.27 1.27)) (justify left))
     )
-    (property "Footprint" "Connector_PinHeader_2.54mm:PinHeader_1x02_P2.54mm_Vertical" (id 2) (at 30.48 61.976 90)
+    (property "Footprint" "meteo_station_footprints:SolarPanel" (id 2) (at 30.48 61.976 90)
       (effects (font (size 1.27 1.27)) hide)
     )
@@
     (property "Reference" "R3" (id 0) (at 154.94 87.63 0))
     (property "Value" "4.7K" (id 1) (at 154.94 85.09 0))
-    (property "Footprint" "Resistor_SMD:R_0603_1608Metric_Pad0.98x0.95mm_HandSolder" (id 2) (at 152.908 86.36 90)
+    (property "Footprint" "Resistor_SMD:R_0603_1608Metric" (id 2) (at 152.908 86.36 90)
       (effects (font (size 1.27 1.27)) hide)
     )
@@
     )
     (path "/23797d9f-2c0e-4299-b2b5-bbbc7f9fdf31"
-      (reference "R2") (unit 1) (value "4.7K") (footprint "Resistor_SMD:R_0603_1608Metric_Pad0.98x0.95mm_HandSolder")
+      (reference "R2") (unit 1) (value "4.7K") (footprint "Resistor_SMD:R_0603_1608Metric")
     )
     (path "/e6ee56a2-86c1-42e9-9f14-cd735802777f"
-      (reference "R3") (unit 1) (value "4.7K") (footprint "Resistor_SMD:R_0603_1608Metric_Pad0.98x0.95mm_HandSolder")
+      (reference "R3") (unit 1) (value "4.7K") (footprint "Resistor_SMD:R_0603_1608Metric")
     )
     (path "/e3bc8b35-8aa9-44ed-b10b-bbd343541f80"
-      (reference "SC1") (unit 1) (value "Solar_Cell") (footprint "Connector_PinHeader_2.54mm:PinHeader_1x02_P2.54mm_Vertical")
+      (reference "SC1") (unit 1) (value "Solar_Cell") (footprint "meteo_station_footprints:SolarPanel")
     )
     (path "/a30bd64c-5664-40ec-b5dc-e115cbdaa123"
-      (reference "SW1") (unit 1) (value "SW_SPDT") (footprint "Button_Switch_THT:SW_Slide_1P2T_CK_OS102011MS2Q")
+      (reference "SW1") (unit 1) (value "SW_SPDT") (footprint "meteo_station_footprints:MTS102")
     )
     (path "/1916a1e3-b413-4657-ae92-e4caf1d88b76"
-      (reference "U1") (unit 1) (value "TP4056") (footprint "meteo_station_footprints:BME280")
+      (reference "U1") (unit 1) (value "TP4056") (footprint "meteo_station_footprints:TP4056")
     )
     (path "/93a49863-00ee-408b-9e67-37bd2abd68da"
